File: sd/v1.4/Fubarino_SD_v14.brd (EAGLE design)
At the start: 71.1 x 25.4 mm, 33 parts, among them IC1 PIC32MX440F256H-80I/PT, IC2 MCP1702T-3302E/MB, J1 MICRO_SD_CARD_SOCKET, J2 M28USEPIN1, J3 M28NOPIN1, J8 UX60A-MB-5ST, Q1 8MHz, Q2 32.768 KHz

Commit message: Updated SVG diagram as per Jacob's suggestion (A8/A7 mistake) Updated reference manual with updated diagram. Updated schematic to 1.4.1, with 5V net renamed to Vout as per Jaocb's suggestion.
Connections:
- net 5V renamed VOUT
Changed lines of the file:
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@@
 <?xml version="1.0" encoding="utf-8"?>
 <!DOCTYPE eagle SYSTEM "eagle.dtd">
-<eagle version="6.2">
+<eagle version="6.4">
 <drawing>
 <settings>
@@
 </class>
 </classes>
-<designrules>
+<designrules name="default">
 <description language="de">&lt;b&gt;EAGLE Design Rules&lt;/b&gt;
 &lt;p&gt;
@@
 <wire x1="25.92" y1="10.06" x2="25.82" y2="10.16" width="0.2032" layer="1"/>
 </signal>
-<signal name="5V">
+<signal name="VOUT">
 <contactref element="IC2" pad="2@1"/>
 <contactref element="IC2" pad="2"/>
