File: accessories/FubarStep/FuabarStep_v10/FubarStep_v10.sch (EAGLE design)
At the start: 54 parts, among them IC2 SN754410NE, IC3 SN754410NE, U1 FUBARINO_SD, U2 FUBARINO_MINI, U3 OKI-78SR-5/1.5-W36H-C, X1 DC21MMX

Commit message: Added power mode jumper to select between 12V and 5V inputs. Added two ground pins for debugging Added 2-pin screw terminal for extra power input option.
Parts:
- added JP3: (no value), SparkFun-Connectors:M03PTH
- added JP4: (no value), SparkFun-Connectors:M023.5MM
- added JP5, JP6: M01PTH, SparkFun-Connectors:M01PTH
Connections:
- new net N$2: JP3.1, U3.OUT
- net +5V: now also JP3.2; no longer U3.OUT
- net GND: now also JP4.1, JP5.1, JP6.1
- net VIN: now also JP3.3, JP4.2
Other:
- note added: "12V DC or 5V DC in"
- note added: "Power Select Jumper 1-2 = 12V in, use regulator 2-3 = 5V in, bypass regulator"
- note removed: "12V DC in (anywhere from 7V to 24V OK)"
Changed lines of the file:
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@@
 <part name="JP34" library="SparkFun-Connectors" deviceset="M03" device="PTH"/>
 <part name="U$1" library="SchmalzHaus" deviceset="SCHMALZHAUS" device="SCHMALZHAUS_SMALL"/>
+<part name="JP3" library="SparkFun-Connectors" deviceset="M03" device="PTH"/>
+<part name="SUPPLY13" library="SparkFun-Aesthetics" deviceset="VIN" device=""/>
+<part name="JP4" library="SparkFun-Connectors" deviceset="M02" device="3.5MM"/>
+<part name="SUPPLY14" library="SparkFun-Aesthetics" deviceset="VIN" device=""/>
+<part name="JP5" library="SparkFun-Connectors" deviceset="M01" device="PTH"/>
+<part name="JP6" library="SparkFun-Connectors" deviceset="M01" device="PTH"/>
+<part name="GND21" library="supply1" deviceset="GND" device=""/>
+<part name="GND22" library="supply1" deviceset="GND" device=""/>
 </parts>
 <sheets>
@@
 <text x="17.78" y="152.4" size="1.778" layer="98">FTDI Serial</text>
 <text x="116.84" y="170.18" size="1.778" layer="98">RC Servo/5V tollerant GPIO</text>
-<text x="7.62" y="99.06" size="1.778" layer="98">Power Supply</text>
-<text x="7.62" y="93.98" size="1.778" layer="98">12V DC in (anywhere from 7V to 24V OK)</text>
+<text x="7.62" y="104.14" size="1.778" layer="98">Power Supply</text>
+<text x="7.62" y="93.98" size="1.778" layer="98">12V DC or 5V DC in</text>
 <text x="7.62" y="241.3" size="1.778" layer="98">chipKIT Fubarino (use only one a time)</text>
 <text x="200.66" y="132.08" size="1.778" layer="98">Analog Input/3.3v only GPIO</text>
@@
 <wire x1="71.12" y1="114.3" x2="71.12" y2="154.94" width="0.1524" layer="98"/>
 <wire x1="71.12" y1="154.94" x2="15.24" y2="154.94" width="0.1524" layer="98"/>
-<wire x1="5.08" y1="101.6" x2="106.68" y2="101.6" width="0.1524" layer="98"/>
-<wire x1="106.68" y1="101.6" x2="106.68" y2="38.1" width="0.1524" layer="98"/>
-<wire x1="106.68" y1="38.1" x2="5.08" y2="38.1" width="0.1524" layer="98"/>
-<wire x1="5.08" y1="38.1" x2="5.08" y2="101.6" width="0.1524" layer="98"/>
+<wire x1="5.08" y1="106.68" x2="111.76" y2="106.68" width="0.1524" layer="98"/>
+<wire x1="111.76" y1="106.68" x2="111.76" y2="25.4" width="0.1524" layer="98"/>
+<wire x1="111.76" y1="25.4" x2="5.08" y2="25.4" width="0.1524" layer="98"/>
+<wire x1="5.08" y1="25.4" x2="5.08" y2="106.68" width="0.1524" layer="98"/>
 <wire x1="114.3" y1="172.72" x2="187.96" y2="172.72" width="0.1524" layer="98"/>
 <wire x1="187.96" y1="172.72" x2="187.96" y2="25.4" width="0.1524" layer="98"/>
@@
 <text x="7.62" y="7.62" size="1.778" layer="98"> software, hardware and materials distributed under this License is distributed on an “AS IS” BASIS, WITHOUT WARRANTIES OR CONDITIONS OF ANY KIND, either express or implied. </text>
 <text x="7.62" y="5.08" size="1.778" layer="98"> See the License for the specific language governing permissions and limitations under the License.</text>
+<text x="66.04" y="96.52" size="1.778" layer="98">Power Select Jumper
+1-2 = 12V in, use regulator
+2-3 = 5V in, bypass regulator</text>
 </plain>
 <instances>
@@
 <instance part="JP34" gate="G$1" x="177.8" y="45.72" rot="R180"/>
 <instance part="U$1" gate="G$1" x="254" y="10.16"/>
+<instance part="JP3" gate="G$1" x="73.66" y="91.44" rot="R270"/>
+<instance part="SUPPLY13" gate="G$1" x="83.82" y="83.82"/>
+<instance part="JP4" gate="G$1" x="12.7" y="83.82"/>
+<instance part="SUPPLY14" gate="G$1" x="35.56" y="86.36" rot="R270"/>
+<instance part="JP5" gate="G$1" x="30.48" y="35.56" rot="R180"/>
+<instance part="JP6" gate="G$1" x="50.8" y="35.56" rot="R180"/>
+<instance part="GND21" gate="1" x="15.24" y="30.48"/>
+<instance part="GND22" gate="1" x="38.1" y="30.48"/>
 </instances>
 <busses>
@@
 <net name="+5V" class="0">
 <segment>
-<pinref part="U3" gate="G$1" pin="OUT"/>
-<wire x1="68.58" y1="71.12" x2="76.2" y2="71.12" width="0.1524" layer="91"/>
 <pinref part="C1" gate="G$1" pin="1"/>
 <wire x1="76.2" y1="71.12" x2="91.44" y2="71.12" width="0.1524" layer="91"/>
 <wire x1="76.2" y1="66.04" x2="76.2" y2="71.12" width="0.1524" layer="91"/>
-<junction x="76.2" y="71.12"/>
 <pinref part="P+1" gate="1" pin="+5V"/>
 <wire x1="91.44" y1="71.12" x2="91.44" y2="76.2" width="0.1524" layer="91"/>
@@
 <pinref part="C5" gate="G$1" pin="+"/>
 <wire x1="91.44" y1="71.12" x2="91.44" y2="66.04" width="0.1524" layer="91"/>
+<pinref part="JP3" gate="G$1" pin="2"/>
+<wire x1="73.66" y1="83.82" x2="73.66" y2="71.12" width="0.1524" layer="91"/>
+<wire x1="73.66" y1="71.12" x2="76.2" y2="71.12" width="0.1524" layer="91"/>
+<junction x="76.2" y="71.12"/>
 </segment>
 <segment>
@@
 <pinref part="GND19" gate="1" pin="GND"/>
 <pinref part="X1" gate="G$1" pin="3"/>
+<pinref part="JP4" gate="G$1" pin="1"/>
+<wire x1="20.32" y1="83.82" x2="35.56" y2="83.82" width="0.1524" layer="91"/>
+<wire x1="35.56" y1="83.82" x2="35.56" y2="71.12" width="0.1524" layer="91"/>
+<junction x="35.56" y="71.12"/>
 </segment>
 <segment>
@@
 <junction x="165.1" y="88.9"/>
 </segment>
+<segment>
+<pinref part="JP5" gate="G$1" pin="1"/>
+<pinref part="GND21" gate="1" pin="GND"/>
+<wire x1="22.86" y1="35.56" x2="15.24" y2="35.56" width="0.1524" layer="91"/>
+<wire x1="15.24" y1="35.56" x2="15.24" y2="33.02" width="0.1524" layer="91"/>
+</segment>
+<segment>
+<pinref part="JP6" gate="G$1" pin="1"/>
+<pinref part="GND22" gate="1" pin="GND"/>
+<wire x1="43.18" y1="35.56" x2="38.1" y2="35.56" width="0.1524" layer="91"/>
+<wire x1="38.1" y1="35.56" x2="38.1" y2="33.02" width="0.1524" layer="91"/>
+</segment>
 </net>
 <net name="VIN" class="0">
@@
 <pinref part="C16" gate="G$1" pin="+"/>
 <wire x1="215.9" y1="165.1" x2="215.9" y2="160.02" width="0.1524" layer="91"/>
+</segment>
+<segment>
+<pinref part="JP3" gate="G$1" pin="3"/>
+<wire x1="76.2" y1="83.82" x2="76.2" y2="81.28" width="0.1524" layer="91"/>
+<wire x1="76.2" y1="81.28" x2="83.82" y2="81.28" width="0.1524" layer="91"/>
+<pinref part="SUPPLY13" gate="G$1" pin="VIN"/>
+<wire x1="83.82" y1="81.28" x2="83.82" y2="83.82" width="0.1524" layer="91"/>
+</segment>
+<segment>
+<pinref part="JP4" gate="G$1" pin="2"/>
+<pinref part="SUPPLY14" gate="G$1" pin="VIN"/>
+<wire x1="20.32" y1="86.36" x2="35.56" y2="86.36" width="0.1524" layer="91"/>
 </segment>
 </net>
@@
 </segment>
 </net>
+<net name="N$2" class="0">
+<segment>
+<pinref part="JP3" gate="G$1" pin="1"/>
+<wire x1="71.12" y1="83.82" x2="71.12" y2="71.12" width="0.1524" layer="91"/>
+<pinref part="U3" gate="G$1" pin="OUT"/>
+<wire x1="71.12" y1="71.12" x2="68.58" y2="71.12" width="0.1524" layer="91"/>
+</segment>
+</net>
 </nets>
 </sheet>
@@
 </schematic>
 </drawing>
+<compatibility>
+<note version="6.3" minversion="6.2.2" severity="warning">
+Since Version 6.2.2 text objects can contain more than one line,
+which will not be processed correctly with this version.
+</note>
+</compatibility>
 </eagle>
