File: sdz/v1.0/Fubarino_SD_v10.sch (EAGLE design)
At the start: 37 parts, among them IC2 MCP1702T-3302E/MB, J1 MICRO_SD_CARD_SOCKET, J2 M28USEPIN1, J3 M28NOPIN1, J8 USB-5PIN, Q1 8MHz, Q2 32.768 KHz

Commit message: More work on FBSDZ
Parts:
- removed C14, C15: 12pF, SparkFun:CAP0603-CAP
- removed J8: USB-5PIN, SchmalzHaus:USB-5PIN
- removed LED1: RED, SparkFun:LED0603
- removed LED2: GREEN, SparkFun:LED0603
- removed PROGRAM, RESET: PTS525SM10SMTR LFS, SparkFun02-20-08:TAC_SWITCHSND
- removed Q1: 8MHz, SchmalzHaus:CRYSTALNX5032
- removed U$6: PIC32MZXXXXECX064TQFP-10X10, SchmalzHaus:PIC32MZXXXXECX064TQFP-10X10
- added D3: GREEN, OPL Eagle Library:LED
- added D4: RED, OPL Eagle Library:LED
- added IC1: PIC32MZXXXXECX064TQFP-10X10, SchmalzHaus:PIC32MZXXXXECX064TQFP-10X10
- added IC3: DSC1033_MICREL_OSCILLATOR3.2X2.5, SchmalzHaus:DSC1033_MICREL_OSCILLATOR3.2X2.5
- added J4: MICRO-USB-5P-340015001, OPL Eagle Library:MICRO-USB-5P-340015001
- added JP1: (no value), SparkFun-Passives:JUMPER-2SMD-NO
- added S1, S2: (no value), SchmalzHaus:SWITCH
- C1, C2, C3, C4, C8, C9: device SparkFun:CAP0603-CAP -> OPL Eagle Library:C-0603
- C10: device SparkFun02-20-08:CAP0603 -> OPL Eagle Library:C-0603
- C13: device SparkFun02-20-08:CAP0805 -> OPL Eagle Library:C-0805
- C5: device SchmalzHaus:CAP0805 -> OPL Eagle Library:C-0805
- R1, R10, R11, R3, R8, R9: device SparkFun:RESISTOR0603-RES -> OPL Eagle Library:R-0603
Connections:
- removed net OSC2: C15.2, Q1.2, U$6.OSCO/CLKO/RC15
- removed net RD6: J2.16
- removed net RD7: J2.17
- removed net RD8: J2.4
- removed net USBID: J8.ID, R9.1, U$6.USBID/PRF3/RF3
- new net RC15: IC1.OSCO/CLKO/RC15, J2.16
- new net USBID/RF3: IC1.USBID/PRF3/RF3, J2.17, J4.ID, R9.1
- net !MCLR!: now also IC1.!MCLR!, S2.2; no longer RESET.3, RESET.4, U$6.!MCLR!
- net 3.3V: now also IC1.AVDD, IC1.VDD@1, IC1.VDD@3, IC1.VDD@4, IC1.VDD@5, IC1.VDD@6, IC3.VDD; no longer U$6.AVDD, U$6.VDD@1, U$6.VDD@3, U$6.VDD@4, U$6.VDD@5, U$6.VDD@6
- net 5V: now also JP1.2
- net D+: now also IC1.D+, J4.DP; no longer J8.D+, U$6.D+
- net D-: now also IC1.D-, J4.DM; no longer J8.D-, U$6.D-
- net GND: now also D4.-, IC1.AVSS, IC1.VSS@1, IC1.VSS@2, IC1.VSS@3, IC1.VSS@4, IC1.VSS@5, IC1.VSS@6, IC3.GND, J4.GND@1, J4.GND@2, J4.GND@3, S1.1, S2.1; no longer C14.1, C15.1, J8.GND, J8.MTN1, J8.MTN2, J8.MTN3, J8.MTN4, LED1.C, PROGRAM.1, PROGRAM.2, RESET.1, RESET.2, U$6.AVSS, U$6.VSS@1, U$6.VSS@2, U$6.VSS@3, U$6.VSS@4, U$6.VSS@5, U$6.VSS@6
- net N$110: now also IC1.VUSB3V3; no longer U$6.VUSB3V3
- net N$20: now also D3.-; no longer LED2.C
- net N$6: now also D4.+; no longer LED1.A
- net OSC1: now also IC1.OSCI/CLKI/RC12, IC3.OUT; no longer C14.2, Q1.1, U$6.OSCI/CLKI/RC12
- net RB0: now also IC1.PGED1/VREF+/CVREF+/AN0/RPB0/PMA6/RB0; no longer U$6.PGED1/VREF+/CVREF+/AN0/RPB0/PMA6/RB0
- net RB1: now also IC1.PGEC1/VREF-/CVREF-/AN1/RPB1/RB1; no longer U$6.PGEC1/VREF-/CVREF-/AN1/RPB1/RB1
- net RB10: now also IC1.TMS/CVREFOUT/AN5/RPB10/PMA13/RB10; no longer U$6.TMS/CVREFOUT/AN5/RPB10/PMA13/RB10
- net RB11: now also IC1.TDO/AN6/PMA12/RB11; no longer U$6.TDO/AN6/PMA12/RB11
- net RB12: now also IC1.TCK/AN7/PMA11/RB12; no longer U$6.TCK/AN7/PMA11/RB12
- net RB13: now also IC1.TDI/AN8/RB13; no longer U$6.TDI/AN8/RB13
- net RB14: now also IC1.AN9/RPB14/SCK3/PMA1/RB14; no longer U$6.AN9/RPB14/SCK3/PMA1/RB14
- net RB15: now also IC1.AN10/EMDC/AEMDC/RPB15/OCFB/PMA0/RB15; no longer U$6.AN10/EMDC/AEMDC/RPB15/OCFB/PMA0/RB15
- net RB2: now also IC1.AN2/C2INB/RPB2/RB2; no longer U$6.AN2/C2INB/RPB2/RB2
- net RB3: now also IC1.AN3/C2INA/RPB3/RB3; no longer U$6.AN3/C2INA/RPB3/RB3
- net RB4: now also IC1.AN4/C1INB/RB4; no longer U$6.AN4/C1INB/RB4
- net RB5: now also IC1.AN45/C1INA/RPB5/RB5, J2.4; no longer U$6.AN45/C1INA/RPB5/RB5
- net RB6: now also IC1.PGEC2/AN46/RPB6/RB6; no longer U$6.PGEC2/AN46/RPB6/RB6
- net RB7: now also IC1.PGED2/AN7/RPB7/RB7; no longer U$6.PGED2/AN7/RPB7/RB7
- net RB8: now also IC1.AN48/RPB8/PMA10/RB8; no longer U$6.AN48/RPB8/PMA10/RB8
- net RB9: now also IC1.AN49/RPB9/PMA7/RB9; no longer U$6.AN49/RPB9/PMA7/RB9
- net RC13: now also IC1.SOSCI/RPC13/RC13; no longer U$6.SOSCI/RPC13/RC13
- net RC14: now also IC1.SOSCO/RPC14/T1CK/RC14; no longer U$6.SOSCO/RPC14/T1CK/RC14
- net RD0: now also IC1.AERXD1/ETXD3/RPD0/RTCC/INT0/RD0; no longer U$6.AERXD1/ETXD3/RPD0/RTCC/INT0/RD0
- net RD1: now also IC1.EMDIO/AEMDIO/RPD1/SCK1/RD1; no longer U$6.EMDIO/AEMDIO/RPD1/SCK1/RD1
- net RD10: now also IC1.ECOL/RPD10/SCL1/SCK4/RD10; no longer U$6.ECOL/RPD10/SCL1/SCK4/RD10
- net RD11: now also IC1.AERXCLK/AEREFCLK/ECRS/RPD11/PMCS1/PMA14/RD11; no longer U$6.AERXCLK/AEREFCLK/ECRS/RPD11/PMCS1/PMA14/RD11
- net RD2: now also IC1.ETXERR/AETXEN/RPD2/SDA3/RD2; no longer U$6.ETXERR/AETXEN/RPD2/SDA3/RD2
- net RD3: now also IC1.AERXERR/ETXCLK/RPD3/SCL3/RD3; no longer U$6.AERXERR/ETXCLK/RPD3/SCL3/RD3
- net RD4: now also IC1.!SQICS0!/RPD4/PMWR/RD4; no longer U$6.!SQICS0!/RPD4/PMWR/RD4
- net RD5: now also IC1.!SQICS1!/RPD5/PMRD/RD5; no longer U$6.!SQICS1!/RPD5/PMRD/RD5
- net RD9: now also IC1.AERXD0/ETXD2/RPD9/SDA1/PMCS2/PMA15/RD9; no longer U$6.AERXD0/ETXD2/RPD9/SDA1/PMCS2/PMA15/RD9
- net RE0: now also IC1.TRD0/SQID0/ERXD1/PMD0/RE0; no longer U$6.TRD0/SQID0/ERXD1/PMD0/RE0
- net RE1: now also IC1.TRD1/SQID1/ERXD0/PMD1/RE1; no longer U$6.TRD1/SQID1/ERXD0/PMD1/RE1
- net RE2: now also IC1.TRD2/EQID2/ERXDV/ECRSDV/AECRSDVPMD2/RE2; no longer U$6.TRD2/EQID2/ERXDV/ECRSDV/AECRSDVPMD2/RE2
- net RE3: now also IC1.TRD3/SQID3/ERXCLK/EREFCLK/RPE3/PMD3/RE3; no longer U$6.TRD3/SQID3/ERXCLK/EREFCLK/RPE3/PMD3/RE3
- net RE4: now also IC1.AN18/ERXERR/PMD4/RE4; no longer U$6.AN18/ERXERR/PMD4/RE4
- net RE5: now also D3.+, IC1.AN17/ETXEN/RPE5/PMD5/RE5; no longer LED2.A, U$6.AN17/ETXEN/RPE5/PMD5/RE5
- net RE6: now also IC1.AN16/ETXD0/PMD6/RE6; no longer U$6.AN16/ETXD0/PMD6/RE6
- net RE7: now also IC1.AN15/ETXD1/PMD7/RE7, S1.2; no longer PROGRAM.3, PROGRAM.4, U$6.AN15/ETXD1/PMD7/RE7
- net RF0: now also IC1.ERXD3/AETXD1/RPF0/RF0; no longer U$6.ERXD3/AETXD1/RPF0/RF0
- net RF1: now also IC1.TRCLK/SQICLK/ERXD2/AETXD0/RPF1/RF1; no longer U$6.TRCLK/SQICLK/ERXD2/AETXD0/RPF1/RF1
- net RF4: now also IC1.RPF4/SDA5/PMA9/RF4; no longer U$6.RPF4/SDA5/PMA9/RF4
- net RF5: now also IC1.RPF5/SCL5/PMA8/RF5; no longer U$6.RPF5/SCL5/PMA8/RF5
- net RG6: now also IC1.AN14/C1IND/RPG6/SCK2/PMA5/RG6; no longer U$6.AN14/C1IND/RPG6/SCK2/PMA5/RG6
- net RG7: now also IC1.AN13/C1INC/RPG7/SDA4/PMA4/RG7; no longer U$6.AN13/C1INC/RPG7/SDA4/PMA4/RG7
- net RG8: now also IC1.AN12/C2IND/RPG8/SCL4/PMA3/RG8; no longer U$6.AN12/C2IND/RPG8/SCL4/PMA3/RG8
- net RG9: now also IC1.AN11/C2INC/RPG9/PMA2/RG9; no longer U$6.AN11/C2INC/RPG9/PMA2/RG9
- net VBUS: now also IC1.VBUS, J4.VCC, JP1.1; no longer J8.VBUS, U$6.VBUS
Other:
- note added: "Apply 5V to VIN or VOUT and connect JP1 for USB host"
- note added: "PRG"
- note added: "Power ON LED (RED)"
- note added: "User LED (GREEN) Blinks when in bootloader mode"
- note removed: "Power ON LED"
- moved on the sheet: J2, J3, Q2

Commit message: This version got sent to seed for fab - v 1.0
Parts:
- added C6: 0.1uF, OPL Eagle Library:C-0603
- added J5: MICRO-SDCARD-CONNECTOR-3300060P1, OPL Eagle Library:MICRO-SDCARD-CONNECTOR-3300060P1
- added R2: 1K, OPL Eagle Library:R-0603
Connections:
- new net $MCLR: C6.1, R10.2, R2.1, S2.2
- net !MCLR!: now also R2.2; no longer R10.2, S2.2
- net 3.3V: now also J5.VDD
- net GND: now also C6.2, J5.G1, J5.G2, J5.G3, J5.G4, J5.VSS
- net RG6: now also J5.SCLK
- net RG7: now also J5.DO
- net RG8: now also J5.DI
- net RG9: now also J5.CS
Other:
- moved on the sheet: C10, C13, C3, C8, C9, D1, D2, D3, D4, IC2, J4, JP1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
