File: mini/v17/FubarinoMini_v17.brd (EAGLE design)
At the start: 50.8 x 17.8 mm, 36 parts, among them IC1 MCP1702T-3302E/MB, J1 M20, J2 M20, J8 USB-5PIN, Q1 8MHz, Q2 32.768 KHz, U1 PIC32MX250F128D_44VTLA_44

Commit message: Updated design to final v1.7 - see Notes.txt for change list
Parts:
- D1, D2: value B0540WS-7 -> CUS15S40,H3F
- IC1: value MCP1702T-3302E/MB -> AP7215-33YG-13
- R11, R8: value 330 -> 820
- U1: value PIC32MX250F128D_44VTLA_44 -> PIC32MX270F256D_44QFN_44
Other:
- board text added: "Copyright 2012-2018 Brian Schmalz Copyright and related rights are licensed under the Solderpad Hardware License, Version 0.51 (the “License”);"
- board text added: "TITLE: FUBARINO MINI VERSION: 1.7 DATE: 5/02/2018 PCB DESIGNER: BRIAN SCHMALZ ENGINEER: BRIAN SCHMALZ"
- board text removed: "Copyright 2012 Brian Schmalz Copyright and related rights are licensed under the Solderpad Hardware License, Version 0.51 (the “License”);"
- board text removed: "TITLE: FUBARINO MINI VERSION: 1.6 DATE: 3/14/2013 PCB DESIGNER: BRIAN SCHMALZ ENGINEER: BRIAN SCHMALZ"

Commit message: Changed LDO to one that has 15V VIn max. Still need to updated caps on either side to be bigger.
Parts:
- IC1: value AP7215-33YG-13 -> AZ1117CR2-3.3TRG1
Changed lines of the file:
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@@
 <?xml version="1.0" encoding="utf-8"?>
 <!DOCTYPE eagle SYSTEM "eagle.dtd">
-<eagle version="9.0.0">
+<eagle version="8.7.1">
 <drawing>
 <settings>
@@
 <attribute name="VALUE" x="-2.4384" y="13.2842" size="0.6096" layer="27"/>
 </element>
-<element name="IC1" library="linear" package="SOT89" value="AP7215-33YG-13" x="37.4904" y="11.7348" smashed="yes" rot="R270">
+<element name="IC1" library="linear" package="SOT89" value="AZ1117CR2-3.3TRG1" x="37.4904" y="11.7348" smashed="yes" rot="R270">
 <attribute name="NAME" x="37.1348" y="13.843" size="0.6096" layer="25"/>
 <attribute name="VALUE" x="35.0345" y="14.6035" size="0.6096" layer="27"/>
